Commit message: URDF: add base_link->imu_link fixed joint (BNO085 mount, S30)
Measured offset xyz=(-0.0165,-0.002,0.055), rpy=0. Flat mount; in-plane pose irrelevant to the yaw-rate signal. Completes TF tree ahead of the EKF.

Co-Authored-By: Claude Opus 4.8 <noreply@anthropic.com>

Claude-Session: https://claude.ai/code/session_01L1RCW2ztsVsWxEkQAjFXAZ

File: picarx_ros/urdf/picarx.urdf (robot description, URDF)
Before this commit: robot picarx, 2 links, 1 joints
Links:
- added link imu_link; visual box size=0.020 0.018 0.003
Joints:
- added joint base_to_imu: type fixed, parent base_link, child imu_link, origin xyz=-0.0165 -0.002 0.055 rpy=0 0 0
